File: HARDWARE/unified_control_board/unified_control_board.kicad_pcb (KiCad board)
At the start: 4 copper layers, 100 x 100 mm, 142 parts, among them J1 Conn_01x03, J10 Conn_01x03, J11 Conn_01x03, J12 Conn_01x03, J13 Conn_01x03, J14 Conn_01x03, J15 Conn_01x03, J16 Conn_01x03, J17 Conn_01x03, J18 Conn_01x03, J19 Conn_01x03, J2 Conn_01x03, J20 Conn_01x03, J21 Conn_01x03, J22 Conn_01x03, J23 Conn_01x03, J24 Conn_01x03, J25 Conn_01x03, J26 Conn_01x03, J27 Conn_01x03, J28 Conn_01x03, J29 Conn_01x03, J3 Conn_01x03, J30 Conn_01x03, J31 Conn_01x03, J32 Conn_01x03, J33 Screw Terminal, J34 ICSP, J35 Conn_01x03, J36 Conn_01x02, J4 Conn_01x03, J5 Conn_01x03, J6 Conn_01x03, J7 Conn_01x03, J8 Conn_01x03, J9 Conn_01x03, Q1 Q_NMOS_DGS, Q10 Q_NMOS_DGS, Q11 Q_NMOS_DGS, Q12 Q_NMOS_DGS, Q13 Q_NMOS_DGS, Q14 Q_NMOS_DGS, Q15 Q_NMOS_DGS, Q16 Q_NMOS_DGS, Q17 Q_NMOS_DGS, Q18 Q_NMOS_DGS, Q19 Q_NMOS_DGS, Q2 Q_NMOS_DGS, Q20 Q_NMOS_DGS, Q21 Q_NMOS_DGS, Q22 Q_NMOS_DGS, Q23 Q_NMOS_DGS, Q24 Q_NMOS_DGS, Q25 Q_NMOS_DGS, Q26 Q_NMOS_DGS, Q27 Q_NMOS_DGS, Q28 Q_NMOS_DGS, Q29 Q_NMOS_DGS, Q3 Q_NMOS_DGS, Q30 Q_NMOS_DGS, Q31 Q_NMOS_DGS, Q32 Q_NMOS_DGS, Q33 Q_NMOS_DGS, Q4 Q_NMOS_DGS, Q5 Q_NMOS_DGS, Q6 Q_NMOS_DGS, Q7 Q_NMOS_DGS, Q8 Q_NMOS_DGS, Q9 Q_NMOS_DGS, SW1 SW_Push, U1 ATmega2560-16A, U2 NCA9306DCH, U3 MCP1825S-500, U4 MCP1824ST-330, Y1 16MHz

Commit message: v1.0 of unified control board
Parts:
- removed RN13: 4.7kΩ, Resistor_SMD:R_Array_Convex_2x0603
- added G***: LOGO, logo:arc_logo, F.Cu at (77.8, 122.5)
- U2: value NCA9306DCH -> RS0102YH8; footprint level_shifter:SOP50P310X100-8N -> Package_TO_SOT_SMD:SOT-23-8
- moved C13 6.58 mm to (75.8, 93.2), turned to -90 degrees
- moved C14 5.73 mm to (75.8, 97.8), turned to 90 degrees
- moved U2 3.04 mm to (72.2, 95.5), turned to -90 degrees
- moved G*** 1.52 mm to (64.8, 119.5)
- moved RN7 0.25 mm to (32.8, 81.2)
Connections:
- C13 pad 1: +3V3 -> GND
- C13 pad 2: GND -> VDD
- C14 pad 2: VDD -> +3V3
- J35 pad 1: /SDA_3.3v -> /RxD_3v3
- J35 pad 2: /SCL_3.3v -> /TxD_3v3
- U1 pad 43: /SCL -> unconnected-(U1-PD0-Pad43)
- U1 pad 44: /SDA -> unconnected-(U1-PD1-Pad44)
- U1 pad 45: unconnected-(U1-PD2-Pad45) -> /RxD
- U1 pad 46: unconnected-(U1-PD3-Pad46) -> /TxD
- U2 pad 1: GND -> VDD
- U2 pad 2: +3V3 -> /RxD
- U2 pad 3: /SCL_3.3v -> /TxD
- U2 pad 4: /SDA_3.3v -> +3V3
- U2 pad 5: /SDA -> GND
- U2 pad 6: /SCL -> /TxD_3v3
- U2 pad 7: VDD -> /RxD_3v3
- U2 pad 8: VDD -> +3V3
Routing:
- net /TxD: track 0.00 -> 26.1 mm, vias 0 -> 2
- net /SCL: track 25.9 -> 0.00 mm, vias 2 -> 0
- net /RxD: track 0.00 -> 25.6 mm, vias 0 -> 2
- net /SDA: track 25.6 -> 0.00 mm, vias 2 -> 0
- net /RST: track 68.0 -> 82.1 mm
- net /TxD_3v3: track 0.00 -> 13.0 mm
- net /RxD_3v3: track 0.00 -> 9.78 mm
- net /SCL_3.3v: track 7.61 -> 0.00 mm
- net /FAN: track 19.5 -> 26.0 mm
- net /SDA_3.3v: track 3.15 -> 0.00 mm
- net +3V3: track 12.1 -> 15.1 mm, vias 2 -> 3
- net VDD: track 30.5 -> 27.9 mm
- net /PWM32: track 91.3 -> 89.4 mm
- net /PWM31: track 85.0 -> 83.2 mm
- net /PWM30: track 78.6 -> 77.0 mm
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- added copper zone on B.Cu, net GND
Other:
- board text added: "32-Channel Servo Driver 10A max per channel 110A max combined"
- board text added: "FAN"
- board text added: "ICSP"
- board text added: "JLCJLCJLCJLC"
- board text added: "Power"
- board text added: "Reset"
- board text added: "Rx"
- board text added: "Tx"
- board text added: "UART"
- board text added: "Wings up!"
- board text removed: "+6V"
- board text removed: "JLCJLCJLC"
