File: HARDWARE/unified_control_board/unified_control_board.kicad_sch (KiCad schematic)
At the start: 137 parts, among them J1 Conn_01x03, J10 Conn_01x03, J11 Conn_01x03, J12 Conn_01x03, J13 Conn_01x03, J14 Conn_01x03, J15 Conn_01x03, J16 Conn_01x03, J17 Conn_01x03, J18 Conn_01x03, J19 Conn_01x03, J2 Conn_01x03, J20 Conn_01x03, J21 Conn_01x03, J22 Conn_01x03, J23 Conn_01x03, J24 Conn_01x03, J25 Conn_01x03, J26 Conn_01x03, J27 Conn_01x03, J28 Conn_01x03, J29 Conn_01x03, J3 Conn_01x03, J30 Conn_01x03, J31 Conn_01x03, J32 Conn_01x03, J33 Screw Terminal, J34 ICSP, J35 Conn_01x03, J36 Conn_01x02, J4 Conn_01x03, J5 Conn_01x03, J6 Conn_01x03, J7 Conn_01x03, J8 Conn_01x03, J9 Conn_01x03, Q1 Q_NMOS_DGS, Q10 Q_NMOS_DGS, Q11 Q_NMOS_DGS, Q12 Q_NMOS_DGS, Q13 Q_NMOS_DGS, Q14 Q_NMOS_DGS, Q15 Q_NMOS_DGS, Q16 Q_NMOS_DGS, Q17 Q_NMOS_DGS, Q18 Q_NMOS_DGS, Q19 Q_NMOS_DGS, Q2 Q_NMOS_DGS, Q20 Q_NMOS_DGS, Q21 Q_NMOS_DGS, Q22 Q_NMOS_DGS, Q23 Q_NMOS_DGS, Q24 Q_NMOS_DGS, Q25 Q_NMOS_DGS, Q26 Q_NMOS_DGS, Q27 Q_NMOS_DGS, Q28 Q_NMOS_DGS, Q29 Q_NMOS_DGS, Q3 Q_NMOS_DGS, Q30 Q_NMOS_DGS, Q31 Q_NMOS_DGS, Q32 Q_NMOS_DGS, Q33 Q_NMOS_DGS, Q4 Q_NMOS_DGS, Q5 Q_NMOS_DGS, Q6 Q_NMOS_DGS, Q7 Q_NMOS_DGS, Q8 Q_NMOS_DGS, Q9 Q_NMOS_DGS, SW1 SW_Push, U1 ATmega2560-16A, U2 NCA9306DCH, U3 MCP1825S-500, U4 MCP1824ST-330, Y1 16MHz

Commit message: Routed PCB
Parts:
- added H1, H2, H3, H4: MountingHole, MountingHole:MountingHole_2.2mm_M2, symbol Mechanical:MountingHole
Connections:
- net ENA17: now also U1.2 (PE0); no longer U1.12 (PH0)
- net ENA18: now also U1.3 (PE1); no longer U1.13 (PH1)
- net ENA19: now also U1.4 (PE2); no longer U1.14 (PH2)
- net ENA20: now also U1.5 (PE3); no longer U1.15 (PH3)
- net ENA21: now also U1.6 (PE4); no longer U1.16 (PH4)
- net ENA22: now also U1.7 (PE5); no longer U1.17 (PH5)
- net ENA23: now also U1.8 (PE6); no longer U1.18 (PH6)
- net ENA24: now also RN3.9 (R8.2), U1.9 (PE7); no longer U1.27 (PH7)
- net ENA25: now also U1.12 (PH0); no longer U1.97 (PF0)
- net ENA26: now also U1.13 (PH1); no longer U1.96 (PF1)
- net ENA27: now also U1.14 (PH2); no longer U1.95 (PF2)
- net ENA28: now also U1.15 (PH3); no longer U1.94 (PF3)
- net ENA29: now also U1.16 (PH4); no longer U1.93 (PF4)
- net ENA30: now also U1.17 (PH5); no longer U1.92 (PF5)
- net ENA31: now also U1.18 (PH6); no longer U1.91 (PF6)
- net ENA32: now also U1.27 (PH7); no longer U1.90 (PF7)
- net FAN: now also U1.23 (PB4); no longer U1.19 (PB0)
- net GND: now also J35.3 (Pin_3); no longer J35.2 (Pin_2)
- net PWM17: now also U1.97 (PF0); no longer U1.89 (PK0)
- net PWM18: now also U1.96 (PF1); no longer U1.88 (PK1)
- net PWM19: now also U1.95 (PF2); no longer U1.87 (PK2)
- net PWM20: now also U1.94 (PF3); no longer U1.86 (PK3)
- net PWM21: now also U1.93 (PF4); no longer U1.85 (PK4)
- net PWM22: now also U1.92 (PF5); no longer U1.84 (PK5)
- net PWM23: now also U1.91 (PF6); no longer U1.83 (PK6)
- net PWM24: now also U1.90 (PF7); no longer RN3.9 (R8.2), U1.82 (PK7)
- net PWM25: now also U1.89 (PK0); no longer U1.2 (PE0)
- net PWM26: now also U1.88 (PK1); no longer U1.3 (PE1)
- net PWM27: now also U1.87 (PK2); no longer U1.4 (PE2)
- net PWM28: now also U1.86 (PK3); no longer U1.5 (PE3)
- net PWM29: now also U1.85 (PK4); no longer U1.6 (PE4)
- net PWM30: now also U1.84 (PK5); no longer U1.7 (PE5)
- net PWM31: now also U1.83 (PK6); no longer U1.8 (PE6)
- net PWM32: now also U1.82 (PK7); no longer U1.9 (PE7)
- net SDA_3.3v: now reaches J35.1 (Pin_1), U2.4 (SDAA)
- net SCL_3.3v: now reaches U2.3 (SCLA)
- net SCL_3.3v: now also J35.2 (Pin_2); no longer J35.3 (Pin_3)
Other:
- moved on the sheet: C1, C10, C11, C12, C13, C14, C2, C3, C4, C5, C6, C7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

Commit message: v1.0 of unified control board
Parts:
- removed RN13: 4.7kΩ, symbol Device:R_Pack02_Split
- removed U2: NCA9306DCH, level_shifter:SOP50P310X100-8N, symbol level_shifter:NCA9306DCH
- added U2: RS0102YH8, SOT-8-RS0102YH8_JRT, symbol level_shifter:RS0102YH8
Connections:
- net +3V3: now also C14.2, U2.4 (OE), U2.8 (VCCA); no longer C13.1
- net GND: now also C13.1, U2.5 (GND); no longer C13.2
- net VDD: now also C13.2, U2.1 (VCCB); no longer C14.2
- net RxD: now reaches U1.45 (PD2)
- net RxD: now also U2.2 (B1)
- net TxD: now reaches U1.46 (PD3)
- net TxD: now also U2.3 (B2)
- net SCL: no longer names the net of U1.43 (PD0)
- net SCL_3.3v renamed TxD_3v3
- net TxD_3v3: now also U2.6 (A2)
- net SDA: no longer names the net of U1.44 (PD1)
- net SDA_3.3v renamed RxD_3v3
- net RxD_3v3: now also U2.7 (A1)
Other:
- moved on the sheet: C13, C14, J35
